File: PCB/FPGA.kicad_sch (KiCad schematic)
At the start: 26 parts, among them U4 LFE5U-12-TG144, U6 UGA

Commit message: WIP
Signed-off-by: Alexis Jeandet <alexis.jeandet@member.fsf.org>
Connections:
- net FPGA_BANK6_IO10 renamed FPGA_IO2
- net FPGA_BANK6_IO11 renamed FPGA_IO1
- net FPGA_BANK6_IO12 renamed FPGA_IO0
- net FPGA_BANK6_IO13: no longer names the net of U4.35 (PL47B/-/HS/LDQ44)
- net FPGA_BANK6_IO14: no longer names the net of U4.37 (PL47C/+/LDQ44/LLC_GPLL0T_IN)
- net FPGA_BANK6_IO6 renamed FPGA_NL
- net FPGA_BANK6_IO7 renamed FPGA_IO5
- net FPGA_BANK6_IO8 renamed FPGA_IO4
- net FPGA_BANK6_IO9 renamed FPGA_IO3

Commit message: release 1.0 ready for production
Signed-off-by: Alexis Jeandet <alexis.jeandet@member.fsf.org>
Other:
- company: (none) -> LPP/CNRS
- title: (none) -> Fusion
