File: PCB/Fusion.kicad_pcb (KiCad board)
At the start: 4 copper layers, 91.5 x 52.1 mm, 133 parts, among them J1 Micro_SD_Card_Det_Hirose_DM3AT, J2 Conn_02x20_Odd_Even, J3 DX07S016JA1R1500, J4 Conn_02x07_Odd_Even, J5 Conn_02x16_Odd_Even, J7 Conn_02x08_Odd_Even, SW1 SW_Push, SW2 SW_Push, U1 STM32F723IETx, U2 TLV62568DDC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

Commit message: WIP
Signed-off-by: Alexis Jeandet <alexis.jeandet@member.fsf.org>
Parts:
- removed JP4: SolderJumper_2_Open, Jumper:SolderJumper-2_P1.3mm_Open_TrianglePad1.0x1.5mm
- added C69: 100nF, Capacitor_SMD:C_0402_1005Metric_Pad0.74x0.62mm_HandSolder, B.Cu at (114.2, 59.9)
- added R39: 10k, Resistor_SMD:R_0402_1005Metric_Pad0.72x0.64mm_HandSolder, B.Cu at (104.1, 54.7)
- added R40: 10k, Resistor_SMD:R_0402_1005Metric_Pad0.72x0.64mm_HandSolder, B.Cu at (105.2, 54.1)
- added R41: 10k, Resistor_SMD:R_0402_1005Metric_Pad0.72x0.64mm_HandSolder, B.Cu at (114.2, 61.0)
- added SW3: RESET, Button_Switch_SMD:SW_SPST_TL3342, B.Cu at (95.7, 76.6)
- added SW4: BOOT0, Button_Switch_SMD:SW_SPST_TL3342, B.Cu at (104.2, 95.1)
- added SYM1: Logo_Open_Hardware_Small, Symbol:OSHW-Logo_11.4x12mm_SilkScreen, B.Cu at (83.5, 57.2)
- added SYM2: Logo_Open_Hardware_Small, Symbol:KiCad-Logo2_8mm_SilkScreen, F.Cu at (87.7, 55.2)
Connections:
- C35 pad 1: /FPGA_BANK6_VCCIO -> /#3.3V
- C36 pad 1: /FPGA_BANK6_VCCIO -> /#3.3V
- J2 pad 7: unconnected-(J2-Pin_7-Pad7) -> GND
- J2 pad 8: unconnected-(J2-Pin_8-Pad8) -> GND
- J5 pad 1: /FPGA_BANK6_VCCIO -> /#3.3V
- J5 pad 10: /FPGA/FPGA_BANK6_IO7 -> /UC_GPIO0
- J5 pad 11: /FPGA/FPGA_BANK6_IO6 -> /FPGA/FPGA_BANK6_IO4
- J5 pad 13: /FPGA/FPGA_BANK6_IO4 -> /FPGA/FPGA_BANK6_IO2
- J5 pad 15: /FPGA/FPGA_BANK6_IO2 -> /FPGA/FPGA_BANK6_IO0
- J5 pad 17: /FPGA/FPGA_BANK6_IO0 -> GND
- J5 pad 3: /FPGA/FPGA_BANK6_IO14 -> /SPI5_MISO
- J5 pad 4: /FPGA/FPGA_BANK6_IO13 -> /I2C1_SDA
- J5 pad 5: /FPGA/FPGA_BANK6_IO12 -> /SPI5_SCK
- J5 pad 6: /FPGA/FPGA_BANK6_IO11 -> /I2C1_SCL
- J5 pad 7: /FPGA/FPGA_BANK6_IO10 -> /SPI5_MOSI
- J5 pad 8: /FPGA/FPGA_BANK6_IO9 -> /UC_GPIO1
- J5 pad 9: /FPGA/FPGA_BANK6_IO8 -> /SPI5_NSS
- J7 pad 11: unconnected-(J7-Pin_11-Pad11) -> GND
- J7 pad 12: unconnected-(J7-Pin_12-Pad12) -> GND
- U1 pad 138: unconnected-(U1-PA15-Pad138) -> /FPGA/FPGA_CFG_CS
- U1 pad 164: unconnected-(U1-PB6-Pad164) -> /I2C1_SCL
- U1 pad 165: unconnected-(U1-PB7-Pad165) -> /FPGA/FPGA_NL
- U1 pad 168: unconnected-(U1-PB9-Pad168) -> /I2C1_SDA
- U1 pad 46: unconnected-(U1-PH5-Pad46) -> /SPI5_NSS
- U1 pad 47: /DAC_OUT1 -> /MCU/ADC_HK_2.5V
- U1 pad 50: /FPGA/FPGA_CFG_CS -> /DAC_OUT1
- U1 pad 54: unconnected-(U1-PC4-Pad54) -> /FPGA/FPGA_IO0
- U1 pad 55: unconnected-(U1-PC5-Pad55) -> /FPGA/FPGA_IO1
- U1 pad 56: unconnected-(U1-PB0-Pad56) -> /UC_GPIO0
- U1 pad 57: unconnected-(U1-PB1-Pad57) -> /UC_GPIO1
- U1 pad 59: unconnected-(U1-PF11-Pad59) -> /SPI5_MOSI
- U1 pad 60: unconnected-(U1-PF12-Pad60) -> /FPGA/FPGA_IO2
- U1 pad 63: unconnected-(U1-PF13-Pad63) -> /FPGA/FPGA_IO3
- U1 pad 64: unconnected-(U1-PF14-Pad64) -> /FPGA/FPGA_IO4
- U1 pad 65: unconnected-(U1-PF15-Pad65) -> /FPGA/FPGA_IO5
- U1 pad 83: unconnected-(U1-PH6-Pad83) -> /SPI5_SCK
- U1 pad 84: unconnected-(U1-PH7-Pad84) -> /SPI5_MISO
- U4 pad 16: /FPGA_BANK6_VCCIO -> /#3.3V
- U4 pad 26: /FPGA/FPGA_BANK6_IO6 -> /FPGA/FPGA_NL
- U4 pad 27: /FPGA/FPGA_BANK6_IO7 -> /FPGA/FPGA_IO5
- U4 pad 28: /FPGA/FPGA_BANK6_IO8 -> /FPGA/FPGA_IO4
- U4 pad 30: /FPGA/FPGA_BANK6_IO9 -> /FPGA/FPGA_IO3
- U4 pad 31: /FPGA/FPGA_BANK6_IO10 -> /FPGA/FPGA_IO2
- U4 pad 33: /FPGA/FPGA_BANK6_IO11 -> /FPGA/FPGA_IO1
- U4 pad 34: /FPGA/FPGA_BANK6_IO12 -> /FPGA/FPGA_IO0
- U4 pad 35: /FPGA/FPGA_BANK6_IO13 -> unconnected-(U4E-PL47B/-/HS/LDQ44-Pad35)
- U4 pad 36: /FPGA_BANK6_VCCIO -> /#3.3V
- U4 pad 37: /FPGA/FPGA_BANK6_IO14 -> unconnected-(U4E-PL47C/+/LDQ44/LLC_GPLL0T_IN-Pad37)
Routing:
- net /I2C1_SCL: track 0.00 -> 81.4 mm, vias 0 -> 2
- net /I2C1_SDA: track 0.00 -> 77.4 mm, vias 0 -> 2
- net /FPGA/FPGA_NL: track 0.00 -> 40.8 mm, vias 0 -> 4
- net /FPGA/FPGA_IO5: track 0.00 -> 36.5 mm, vias 0 -> 2
- net /FPGA/FPGA_IO4: track 0.00 -> 35.1 mm, vias 0 -> 2
- net /FPGA_BANK6_VCCIO: track 35.1 -> 0.00 mm, vias 2 -> 0
- net /FPGA/FPGA_IO3: track 0.00 -> 33.5 mm, vias 0 -> 2
- net /FPGA/FPGA_IO2: track 0.00 -> 31.3 mm, vias 0 -> 2
- net /SPI5_SCK: track 0.00 -> 28.0 mm
- net /FPGA/FPGA_IO1: track 0.00 -> 27.8 mm, vias 0 -> 2
- net /SPI5_MISO: track 0.00 -> 26.4 mm
- net /FPGA/FPGA_IO0: track 0.00 -> 26.3 mm, vias 0 -> 2
- net /#2.5V: track 59.2 -> 84.2 mm, vias 5 -> 6
- net /UC_GPIO0: track 0.00 -> 22.0 mm, vias 0 -> 1
- net /FPGA/FPGA_BANK6_IO13: track 21.5 -> 0.00 mm
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- added copper zone on In1.Cu, net GND
Other:
- board text added: "#3.3V"
- board text added: "AI0"
- board text added: "AI1"
- board text added: "AI2"
- board text added: "AI3"
- board text added: "AI4"
- board text added: "AI5"
- board text added: "AO1"
- board text added: "AO2"
- board text added: "BANK0"
- board text added: "BANK0 IO0-IO8"
- board text added: "BANK0 IO1-IO9"
- board text added: "BANK0 VCCIO"
- board text added: "BANK1"
- board text added: "BANK1 IO0 .... IO14"
- board text added: "BANK1 IO1 .... IO15"
- board text added: "BANK6"
- board text added: "BANK7"
- board text added: "BANK7 IO10 .... IO0"
- board text added: "BANK7 IO11 .... IO1"
- board text added: "BOOT0"
- board text added: "BP1"
- board text added: "BP2"
- board text added: "GND"
- board text added: "LED1"
- board text added: "LED2"
- board text added: "RESET"
- board text added: "USB_5V"

Commit message: release 1.0 ready for production
Signed-off-by: Alexis Jeandet <alexis.jeandet@member.fsf.org>
Routing:
- net /#3.3V: track 133.8 -> 132.8 mm
- net /FPGA/FPGA_CFG_CS: track 41.7 -> 42.4 mm
- net GND: vias 11 -> 18
- net /USB_5V: vias 5 -> 4
Other:
- board text added: "Fusion 1.0 LPP (2024)"
