File: PCB/Fusion.kicad_sch (KiCad schematic)
At the start: 13 parts, among them J2 Conn_02x20_Odd_Even, J5 Conn_02x16_Odd_Even, J7 Conn_02x08_Odd_Even

Commit message: WIP
Signed-off-by: Alexis Jeandet <alexis.jeandet@member.fsf.org>
Parts:
- removed JP4: SolderJumper_2_Open, Jumper:SolderJumper-2_P1.3mm_Open_TrianglePad1.0x1.5mm, symbol Jumper:SolderJumper_2_Open
- added SYM1: Logo_Open_Hardware_Small, Symbol:OSHW-Logo_11.4x12mm_SilkScreen, symbol Graphic:Logo_Open_Hardware_Small
- added SYM2: Logo_Open_Hardware_Small, Symbol:KiCad-Logo2_8mm_SilkScreen, symbol Graphic:Logo_Open_Hardware_Small
Connections:
- net FPGA_BANK6_IO6 is gone; now on net FPGA_BANK6_IO4: J5.11 (Pin_11)
- net FPGA_BANK6_VCCIO is gone; now on net #3.3V: J5.1 (Pin_1)
- net FPGA_BANK6_IO0: now also J5.15 (Pin_15); no longer J5.17 (Pin_17)
- net FPGA_BANK6_IO2: now also J5.13 (Pin_13); no longer J5.15 (Pin_15)
- net FPGA_BANK6_IO4: no longer J5.13 (Pin_13)
- net GND: now also J2.7 (Pin_7), J2.8 (Pin_8), J5.17 (Pin_17), J7.11 (Pin_11), J7.12 (Pin_12)
- net FPGA_BANK6_IO10 renamed SPI5_MOSI
- net FPGA_BANK6_IO11 renamed I2C1_SCL
- net FPGA_BANK6_IO12 renamed SPI5_SCK
- net FPGA_BANK6_IO13 renamed I2C1_SDA
- net FPGA_BANK6_IO14 renamed SPI5_MISO
- net FPGA_BANK6_IO7 renamed UC_GPIO0
- net FPGA_BANK6_IO8 renamed SPI5_NSS
- net FPGA_BANK6_IO9 renamed UC_GPIO1
Other:
- sheet FPGA ports: added FPGA_BANK6_IO[0..5], FPGA_IO0, FPGA_IO1, FPGA_IO2, FPGA_IO3, FPGA_IO4, FPGA_IO5, FPGA_NL; removed FPGA_BANK6_IO[0..14]
- sheet MCU ports: added 2.5V, FPGA_IO0, FPGA_IO1, FPGA_IO2, FPGA_IO3, FPGA_IO4, FPGA_IO5, FPGA_NL, I2C1_SCL, I2C1_SDA, SPI5_MISO, SPI5_MOSI, SPI5_NSS, SPI5_SCK, UC_GPIO0, UC_GPIO1; removed none
- moved on the sheet: JP1, JP2, JP3

Commit message: release 1.0 ready for production
Signed-off-by: Alexis Jeandet <alexis.jeandet@member.fsf.org>
Other:
- company: (none) -> LPP/CNRS
- title: (none) -> Fusion
