File: PCB/MCU.kicad_sch (KiCad schematic)
At the start: 76 parts, among them J1 DX07S016JA1R1500, J1 Micro_SD_Card_Det_Hirose_DM3AT, J4 Conn_02x07_Odd_Even, SW1 SW_Push, SW2 SW_Push, U1 STM32F723IETx, U2 USB6B1, U3 MX25L3233FM1, Y201 12MHz

Commit message: WIP
Signed-off-by: Alexis Jeandet <alexis.jeandet@member.fsf.org>
Parts:
- added C69: 100nF, Capacitor_SMD:C_0402_1005Metric_Pad0.74x0.62mm_HandSolder, symbol Device:C
- added R39, R40, R41: 10k, Resistor_SMD:R_0402_1005Metric_Pad0.72x0.64mm_HandSolder, symbol Device:R
- added SW3: RESET, Button_Switch_SMD:SW_SPST_TL3342, symbol Switch:SW_Push
- added SW4: BOOT0, Button_Switch_SMD:SW_SPST_TL3342, symbol Switch:SW_Push
Connections:
- net 3.3V: now also R39.2, R40.2, SW4.1
- net BOOT0: now also SW4.2
- net DAC_OUT1: now also U1.50 (PA4); no longer U1.47 (PA3)
- net FPGA_CFG_CS: now also U1.138 (PA15); no longer U1.50 (PA4)
- net GND: now also C69.2, SW3.2
- net RESET: now also SW3.1
- net I2C1_SCL: now reaches U1.164 (PB6)
- net I2C1_SCL: now also R40.1
- net FPGA_NL: now reaches U1.165 (PB7)
- net I2C1_SDA: now reaches U1.168 (PB9)
- net I2C1_SDA: now also R39.1
- net SPI5_NSS: now reaches U1.46 (PH5)
- net FPGA_IO0: now reaches U1.54 (PC4)
- net FPGA_IO1: now reaches U1.55 (PC5)
- net UC_GPIO0: now reaches U1.56 (PB0)
- net UC_GPIO1: now reaches U1.57 (PB1)
- net SPI5_MOSI: now reaches U1.59 (PF11)
- net FPGA_IO2: now reaches U1.60 (PF12)
- net FPGA_IO3: now reaches U1.63 (PF13)
- net FPGA_IO4: now reaches U1.64 (PF14)
- net FPGA_IO5: now reaches U1.65 (PF15)
- net SPI5_SCK: now reaches U1.83 (PH6)
- net SPI5_MISO: now reaches U1.84 (PH7)
- new net 2.5V: R41.1
- new net ADC_HK_2.5V: C69.1, R41.2, U1.47 (PA3)
Other:
- moved on the sheet: C2, C210, C47, C48, R35, R36, R37

Commit message: release 1.0 ready for production
Signed-off-by: Alexis Jeandet <alexis.jeandet@member.fsf.org>
Other:
- company: (none) -> LPP/CNRS
- title: (none) -> Fusion
Changed lines of the file:
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@@
 	(generator_version "8.0")
 	(paper "A3")
+	(title_block
+		(title "Fusion")
+		(date "2024-03-15")
+		(rev "1.0")
+		(company "LPP/CNRS")
+		(comment 1 "Alexis Jeandet")
+		(comment 2 "CC-BY-SA")
+		(comment 3 "alexis.jeandet@member.fsf.org")
+	)
 	(junction
 		(at 69.215 238.76)
