File: PCB/TLV62568.kicad_sch (KiCad schematic)
At the start: 7 parts, among them U2 TLV62568DDC

Commit message: release 1.0 ready for production
Signed-off-by: Alexis Jeandet <alexis.jeandet@member.fsf.org>
Other:
- company: (none) -> LPP/CNRS
- title: (none) -> Fusion
