File: PCB/power.kicad_sch (KiCad schematic)
At the start: 4 parts, among them U5 NCP718xSN250

Commit message: release 1.0 ready for production
Signed-off-by: Alexis Jeandet <alexis.jeandet@member.fsf.org>
Other:
- title: USB3 Datalogger -> Fusion
Changed lines of the file:
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@@
 	(paper "A4")
 	(title_block
-		(title "USB3 Datalogger")
-		(date "2020-09-21")
-		(rev "1.1")
+		(title "Fusion")
+		(date "2024-03-15")
+		(rev "1.0")
 		(company "LPP/CNRS")
 		(comment 1 "Alexis Jeandet")
