File: AnalogTwo/AnalogIn.kicad_sch (KiCad schematic)
At the start: 1 part

Commit message: AnaloghTwo ready for production
Signed-off-by: Alexis Jeandet <alexis.jeandet@member.fsf.org>
Parts:
- removed R1: R, Resistor_SMD:R_0603_1608Metric_Pad0.98x0.95mm_HandSolder, symbol Device:R
