File: AnalogTwo/AnalogOut.kicad_sch (KiCad schematic)
At the start: 1 part

Commit message: AnaloghTwo ready for production
Signed-off-by: Alexis Jeandet <alexis.jeandet@member.fsf.org>
Parts:
- removed R50: R, Capacitor_SMD:C_0603_1608Metric_Pad1.08x0.95mm_HandSolder, symbol Device:R
