File: AnalogTwo/AnalogTwo.kicad_pcb (KiCad board)
At the start: 4 copper layers, 96 x 106 mm, 150 parts, among them IC1 AD820, IC2 AD820, J1 Conn_02x08_Odd_Even, J10 Conn_Coaxial_Small, J11 Conn_Coaxial_Small, J12 Conn_Coaxial_Small, J13 Conn_Coaxial_Small, J14 Conn_Coaxial_Small, J15 Conn_Coaxial_Small, J16 Conn_Coaxial_Small, J2 Conn_02x16_Odd_Even, J25 Conn_Coaxial_Small, J26 Conn_Coaxial_Small, J27 Conn_Coaxial_Small, J28 Conn_Coaxial_Small, J3 Conn_02x20_Odd_Even, J4 Conn_Coaxial_Small, J5 Conn_Coaxial_Small, J6 Conn_Coaxial_Small, J9 Conn_Coaxial_Small, U1 ADS92x4R, U13 AD5641AKSZ-500RL7, U14 AD5641AKSZ-500RL7, U2 THS4551, U3 THS4551, U4 ADS92x4R, U5 THS4551, U6 THS4551, U7 TPS65130RGE, U8 TPS7A39, U9 TLV7031DBV

Commit message: AnaloghTwo ready for production
Signed-off-by: Alexis Jeandet <alexis.jeandet@member.fsf.org>
Parts:
- removed R1: R, Resistor_SMD:R_0603_1608Metric_Pad0.98x0.95mm_HandSolder
- removed R50: R, Capacitor_SMD:C_0603_1608Metric_Pad1.08x0.95mm_HandSolder
- added REF**: MountingHole_2.5mm_Pad, MountingHole:MountingHole_2.5mm_Pad, F.Cu at (53.0, 131.0)
- added REF**: MountingHole_2.5mm_Pad, MountingHole:MountingHole_2.5mm_Pad, F.Cu at (126.0, 45.0)
- added REF**: MountingHole_2.5mm_Pad, MountingHole:MountingHole_2.5mm_Pad, F.Cu at (126.0, 145.0)
- added REF**: MountingHole_2.5mm_Pad, MountingHole:MountingHole_2.5mm_Pad, F.Cu at (53.0, 59.0)
- moved FB4 9.09 mm to (87.4, 77.3)
Routing:
- net /Power/DCDC/5V_USB: track 17.9 -> 27.1 mm
- net /USB_5V: track 24.0 -> 15.1 mm
- net GND: track 50.1 -> 49.6 mm
- net /Power/LDO/+6V: track 5.99 -> 6.49 mm
- net /#3.3V: vias 2 -> 0

Commit message: Some last minute fixes
Signed-off-by: Alexis Jeandet <alexis.jeandet@member.fsf.org>
Parts:
- removed the REF** at (126.0, 145.0)
- added FB5: FerriteBead, Inductor_SMD:L_Eaton_MCL2012V1, B.Cu at (76.4, 124.5)
- added REF**: OSHW-Logo2_7.3x6mm_SilkScreen, Symbol:OSHW-Logo2_7.3x6mm_SilkScreen, F.Cu at (110.0, 61.0)
- added REF**: KiCad-Logo2_8mm_SilkScreen, Symbol:KiCad-Logo2_8mm_SilkScreen, F.Cu at (115.0, 140.0)
Connections:
- C88 pad 1: /5V -> /Trigger/filt_3.3V
- C89 pad 1: /5V -> /Trigger/filt_3.3V
- D1 pad 2: /5V -> /#3.3V
- FB1 pad 1: /5V -> /#3.3V
- U9 pad 5: /5V -> /Trigger/filt_3.3V
Routing:
- net /#3.3V: track 49.9 -> 80.2 mm, vias 0 -> 3
- net /Trigger/filt_3.3V: track 0.00 -> 11.7 mm, vias 0 -> 1
- net /5V: track 41.4 -> 35.7 mm, vias 17 -> 15
Other:
- board text added: "AnalogTwo V1.0 Laboratory of Plasma Physics"
