File: AnalogTwo/AnalogTwo.kicad_sch (KiCad schematic)
At the start: 22 parts, among them J1 Conn_02x08_Odd_Even, J10 Conn_Coaxial_Small, J11 Conn_Coaxial_Small, J12 Conn_Coaxial_Small, J13 Conn_Coaxial_Small, J14 Conn_Coaxial_Small, J15 Conn_Coaxial_Small, J16 Conn_Coaxial_Small, J2 Conn_02x16_Odd_Even, J25 Conn_Coaxial_Small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

Commit message: AnaloghTwo ready for production
Signed-off-by: Alexis Jeandet <alexis.jeandet@member.fsf.org>
Other:
- moved on the sheet: C1, C2, C3, C4, J1, J10, J11, J12, J13, J14, J15, J16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

Commit message: Some last minute fixes
Signed-off-by: Alexis Jeandet <alexis.jeandet@member.fsf.org>
Other:
- sheet Trigger ports: added 3.3V; removed 5V
Changed lines of the file:
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@@
 		)
 	)
-	(label "5V"
-		(at 285.75 165.1 0)
-		(fields_autoplaced yes)
-		(effects
-			(font
-				(size 1.27 1.27)
-			)
-			(justify left bottom)
-		)
-	)
 	(label "FPGA_BANK0_IO9"
 		(at 200.66 110.49 180)
@@
 		)
 	)
+	(label "#3.3V"
+		(at 285.75 165.1 0)
+		(fields_autoplaced yes)
+		(effects
+			(font
+				(size 1.27 1.27)
+			)
+			(justify left bottom)
+		)
+	)
 	(label "FPGA_BANK1_IO12"
 		(at 257.81 146.05 180)
@@
 			)
 		)
-		(pin "5V" input
-			(at 283.21 170.18 90)
+		(pin "Trig_out" output
+			(at 307.34 189.23 0)
 			(effects
 				(font
@@
 			)
 		)
-		(pin "Trig_out" output
-			(at 307.34 189.23 0)
+		(pin "3.3V" input
+			(at 283.21 170.18 90)
 			(effects
 				(font
