File: AnalogTwo/Trigger.kicad_sch (KiCad schematic)
At the start: 15 parts, among them U9 TLV7031DBV

Commit message: Some last minute fixes
Signed-off-by: Alexis Jeandet <alexis.jeandet@member.fsf.org>
Parts:
- added FB5: FerriteBead, Inductor_SMD:L_Eaton_MCL2012V1, symbol Device:FerriteBead
Connections:
- net 5V renamed filt_3.3V
- net filt_3.3V: now also FB5.2; no longer D1.2 (K), FB1.1
- new net 3.3V: D1.2 (K), FB1.1, FB5.1
Other:
- moved on the sheet: C85, C86, C87, C88, C89, D1, FB1, JP1, R59, R60, R61, R62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
