File: MainBoardPCB/FPGA.kicad_sch (KiCad schematic)
At the start: 33 parts, among them U301 LFE5U-12-TG144, X1 ECS-2520MV-xxx-xx

Commit message: New FPGA only version
Signed-off-by: Alexis Jeandet <alexis.jeandet@member.fsf.org>
Parts:
- removed U301: LFE5U-12-TG144, Package_QFP:TQFP-144_20x20mm_P0.5mm, symbol ecp5-12-tg144:LFE5U-12-TG144
- added C115: 100nF, Capacitor_SMD:C_0603_1608Metric_Pad1.08x0.95mm_HandSolder, symbol Device:C
- added C201, C202, C203, C204, C205, C206, C207, C208: 22nF, Capacitor_SMD:C_0402_1005Metric, symbol Device:C
- added J201: HDMI_A, Connector_Video:HDMI_A_Molex_208658-1001_Horizontal, symbol Connector:HDMI_A
- added J202: Micro_SD_Card_Det_Hirose_DM3AT, Connector_Card:microSD_HC_Hirose_DM3AT-SF-PEJM5, symbol Connector:Micro_SD_Card_Det_Hirose_DM3AT
- added R108, R201, R202, R203, R204, R205: 10k, Resistor_SMD:R_0402_1005Metric_Pad0.72x0.64mm_HandSolder, symbol Device:R
- added U10: IS25LP128F-JBLE, Package_SO:SOIC-8_5.3x5.3mm_P1.27mm, symbol Memory_EEPROM:25LCxxx
- added U203: LFE5U-85F-6BG381x, Package_BGA:Lattice_caBGA-381_17x17mm_Layout20x20_P0.8mm, symbol FPGA_Lattice:LFE5U-85F-6BG381x
- C1, C301, C302, C303, C304, C305, C306, C307, C308, C310, C311, C313, C315, C316, C318: footprint Capacitor_SMD:C_0402_1005Metric -> Capacitor_SMD:C_0402_1005Metric_Pad0.74x0.62mm_HandSolder
- R305, R307: value R -> 0; now fitted
- R306: value R -> 0; now not fitted
- R308, R309: footprint Resistor_SMD:R_0402_1005Metric -> Resistor_SMD:R_0402_1005Metric_Pad0.72x0.64mm_HandSolder
Connections:
- net FPGA_OPT_CLK is gone; now on net FPGA_CLK: X1.3 (OUT)
- net CFG_0: now also U203.U4 (CFG_0)
- net CFG_1: now also U203.T4 (CFG_1)
- net CFG_2: now also U203.R4 (CFG_2)
- net FPGA_BANK0_IO0: now also U203.A4 (PL11A)
- net FPGA_BANK0_IO1: now also U203.A5 (PL11B)
- net FPGA_BANK0_IO2: now also U203.A2 (PL35A)
- net FPGA_BANK0_IO3: now also U203.A3 (PL14C)
- net FPGA_BANK0_IO4: now also U203.B1 (PL35B)
- net FPGA_BANK0_IO5: now also U203.B2 (PL35C)
- net FPGA_BANK0_IO6: now also U203.C1 (PL38A)
- net FPGA_BANK0_IO7: now also U203.C2 (PL35D)
- net FPGA_BANK0_IO8: now also U203.D1 (PL38B)
- net FPGA_BANK0_IO9: now also U203.D2 (PL38C)
- net FPGA_BANK0_VCCIO: now also U203.H6 (VCCIO7), U203.H7 (VCCIO7), U203.J6 (VCCIO7)
- net FPGA_BANK1_IO0: now also U203.A11 (PT63B)
- net FPGA_BANK1_IO1: now also U203.B11 (PT65A)
- net FPGA_BANK1_IO10: now also U203.B6 (PT4B)
- net FPGA_BANK1_IO11: now also U203.C11 (PT65B)
- net FPGA_BANK1_IO12: now also U203.C10 (PT58B)
- net FPGA_BANK1_IO13: now also U203.C9 (PT54A)
- net FPGA_BANK1_IO14: now also U203.C8 (PT15A)
- net FPGA_BANK1_IO15: now also U203.C7 (PT11B)
- net FPGA_BANK1_IO2: now also U203.A10 (PT63A)
- net FPGA_BANK1_IO3: now also U203.B10 (PT60B)
- net FPGA_BANK1_IO4: now also U203.A9 (PT60A)
- net FPGA_BANK1_IO5: now also U203.B9 (PT58A)
- net FPGA_BANK1_IO6: now also U203.A8 (PT18B)
- net FPGA_BANK1_IO7: now also U203.B8 (PT15B)
- net FPGA_BANK1_IO8: now also U203.A7 (PT18A)
- net FPGA_BANK1_IO9: now also U203.A6 (PT4A)
- net FPGA_BANK1_VCCIO: now also U203.F10 (VCCIO0), U203.F9 (VCCIO0)
- net FPGA_BANK6_IO0: now also U203.J4 (PL50A)
- net FPGA_BANK6_IO1: now also U203.J3 (PL50C)
- net FPGA_BANK6_IO2: now also U203.K5 (PL56B)
- net FPGA_BANK6_IO3: now also U203.J5 (PL50B)
- net FPGA_BANK6_IO4: now also U203.L4 (PL56C)
- net FPGA_BANK6_IO5: now also U203.L3 (PL86C)
- net FPGA_BANK7_IO0: now also U203.F1 (PL47B)
- net FPGA_BANK7_IO1: now also U203.G2 (PL47A)
- net FPGA_BANK7_IO10: now also U203.M1 (PL89B)
- net FPGA_BANK7_IO11: now also U203.N1 (PL89D)
- net FPGA_BANK7_IO2: now also U203.G1 (PL47D)
- net FPGA_BANK7_IO3: now also U203.H2 (PL47C)
- net FPGA_BANK7_IO4: now also U203.H1 (PL53C)
- net FPGA_BANK7_IO5: now also U203.J1 (PL53B)
- net FPGA_BANK7_IO6: now also U203.K2 (PL53A)
- net FPGA_BANK7_IO7: now also U203.K1 (PL53D)
- net FPGA_BANK7_IO8: now also U203.L2 (PL86D)
- net FPGA_BANK7_IO9: now also U203.L1 (PL89C)
- net FPGA_BANK7_VCCIO: now also U203.L6 (VCCIO6), U203.L7 (VCCIO6), U203.M6 (VCCIO6)
- net FPGA_CLK: now also U203.C12 (PT71B)
- net GND: now also C115.2, J201.11 (CKS), J201.17 (GND), J201.2 (D2S), J201.5 (D1S), J201.8 (D0S), J201.SH, J202.11 (SHIELD), J202.6 (VSS), R108.1, U10.4 (GND), U203.B14 (GND), U203.B7 (GND), U203.C19 (GND), U203.D4 (GND), U203.F13 (GND), U203.F14 (GND), U203.F7 (GND), U203.F8 (GND), U203.G10 (GND), U203.G11 (GND), U203.G12 (GND), U203.G13 (GND), U203.G14 (GND), U203.G15 (GND), U203.G17 (GND), U203.G4 (GND), U203.G6 (GND), U203.G7 (GND), U203.G8 (GND), U203.G9 (GND), U203.H19 (GND), U203.J10 (GND), U203.J11 (GND), U203.J12 (GND), U203.J14 (GND), U203.J2 (GND), U203.J7 (GND), U203.J9 (GND), U203.K10 (GND), U203.K11 (GND), U203.K12 (GND), U203.K14 (GND), U203.K15 (GND), U203.K6 (GND), U203.K7 (GND), U203.K9 (GND), U203.L10 (GND), U203.L11 (GND), U203.L12 (GND), U203.L9 (GND), U203.M10 (GND), U203.M11 (GND), U203.M12 (GND), U203.M14 (GND), U203.M16 (GND), U203.M2 (GND), U203.M7 (GND), U203.M9 (GND), U203.N14 (GND), U203.N15 (GND), U203.N6 (GND), U203.N7 (GND), U203.P11 (GND), U203.P12 (GND), U203.P13 (GND), U203.P14 (GND), U203.P7 (GND), U203.P8 (GND), U203.R19 (GND), U203.T10 (GND), U203.T11 (GND), U203.T12 (GND), U203.T13 (GND), U203.T14 (GND), U203.T15 (GND), U203.T6 (GND), U203.T7 (GND), U203.T8 (GND), U203.T9 (GND), U203.U10 (GND), U203.U11 (GND), U203.U12 (GND), U203.U13 (GND), U203.U14 (GND), U203.U15 (GND), U203.U6 (GND), U203.U7 (GND), U203.U8 (GND), U203.U9 (GND), U203.V10 (GND), U203.V11 (GND), U203.V12 (GND), U203.V13 (GND), U203.V14 (GND), U203.V15 (GND), U203.V16 (GND), U203.V17 (GND), U203.V18 (GND), U203.V19 (GND), U203.V20 (GND), U203.V5 (GND), U203.V6 (GND), U203.V7 (GND), U203.V8 (GND), U203.V9 (GND), U203.W12 (GND), U203.W15 (GND), U203.W16 (GND), U203.W19 (GND), U203.W20 (GND), U203.W6 (GND), U203.W7 (GND), U203.Y11 (GND), U203.Y12 (GND), U203.Y14 (GND), U203.Y15 (GND), U203.Y16 (GND), U203.Y17 (GND), U203.Y19 (GND), U203.Y5 (GND), U203.Y6 (GND), U203.Y7 (GND), U203.Y8 (GND)
- net LED1: now also U203.D9 (PT20A)
- net LED2: now also U203.D10 (PT56A)
- net JTAG.TDI: now reaches R303.2
- net JTAG.TDI: now also U203.R5 (TDI)
- net JTAG.TDO: now reaches R301.2
- net JTAG.TDO: now also U203.V4 (TDO)
- net JTAG.TCK: now reaches R302.2
- net JTAG.TCK: now also U203.T5 (TCK)
- net JTAG.TMS: now reaches R304.2
- net JTAG.TMS: now also U203.U5 (TMS)
- net #1.1V renamed 1.1V
- net 1.1V: now also U203.H10 (VCC), U203.H11 (VCC), U203.H12 (VCC), U203.H13 (VCC), U203.H8 (VCC), U203.H9 (VCC), U203.J13 (VCC), U203.J8 (VCC), U203.K13 (VCC), U203.K8 (VCC), U203.L13 (VCC), U203.L8 (VCC), U203.M13 (VCC), U203.M8 (VCC), U203.N10 (VCC), U203.N11 (VCC), U203.N12 (VCC), U203.N13 (VCC), U203.N8 (VCC), U203.N9 (VCC)
- net #2.5V renamed 2.5V
- net 2.5V: now also U203.F15 (VCCAUX), U203.F6 (VCCAUX), U203.P15 (VCCAUX), U203.P6 (VCCAUX)
- net #3.3V renamed 3.3V
- net 3.3V: now also C115.1, J202.10 (DET_A), J202.4 (VDD), R201.1, R202.1, R203.1, R204.1, R205.1, U10.8 (VCC), U203.F11 (VCCIO1), U203.F12 (VCCIO1), U203.H14 (VCCIO2), U203.H15 (VCCIO2), U203.J15 (VCCIO2), U203.L14 (VCCIO3), U203.L15 (VCCIO3), U203.M15 (VCCIO3), U203.P10 (VCCIO8), U203.P9 (VCCIO8)
- new net: R201.2, U10.3 (~{WP})
- new net: R202.2, U10.7 (~{HOLD})
- new net: R203.2, U203.Y3 (DONE)
- new net CARD_DETECT: J202.9 (DET_B), R108.2, U203.U17 (PR92B)
- new net EXT_I²C.SCL: U203.P2 (PL92B)
- new net EXT_I²C.SDA: U203.N4 (PL83C)
- new net EXT_SPI.MISO: U203.N5 (PL83B)
- new net EXT_SPI.MOSI: U203.N3 (PL86A)
- new net EXT_SPI.NSS: U203.M5 (PL77A)
- new net EXT_SPI.SCK: U203.P1 (PL92A)
- new net FLASH_MISO: U10.2 (MISO), U203.V2 (PB11A)
- new net FLASH_MOSI: U10.5 (MOSI), U203.W2 (PB11B)
- new net FLASH_SCK: U10.6 (SCK), U203.U3 (CCLK)
- new net FLASH_nCS: U10.1 (~{CS}), U203.U2 (PB13B)
- new net HDMI_CK+: C208.1, U203.N17 (PR56A)
- new net HDMI_CK-: C207.1, U203.P16 (PR56B)
- new net HDMI_D0+: C206.1, U203.L16 (PR50A)
- new net HDMI_D0-: C205.1, U203.L17 (PR50B)
- new net HDMI_D1+: C204.1, U203.K16 (PR29A)
- new net HDMI_D1-: C203.1, U203.K17 (PR29B)
- new net HDMI_D2+: C201.1, U203.H18 (PR20A)
- new net HDMI_D2-: C202.1, U203.H17 (PR20B)
- new net SDMMC_CLK: J202.5 (CLK), U203.R17 (PR56D)
- new net SDMMC_CMD: J202.3 (CMD), U203.J16 (PR20D)
- new net SDMMC_D0: J202.7 (DAT0), U203.T17 (PR92D)
- new net SDMMC_D1: J202.8 (DAT1), U203.U18 (PR92A)
- new net SDMMC_D2: J202.1 (DAT2), U203.G18 (PR17B)
- new net SDMMC_D3: J202.2 (DAT3/CD), U203.H16 (PR17D)
- new net SDRAM.A0: U203.C16 (PT112A)
- new net SDRAM.A1: U203.C15 (PT105B)
- new net SDRAM.A10: U203.C17 (PT114B)
- new net SDRAM.A11: U203.B18 (PT116B)
- new net SDRAM.A12: U203.A19 (PT121A)
- new net SDRAM.A2: U203.C14 (PT83B)
- new net SDRAM.A3: U203.C13 (PT78B)
- new net SDRAM.A4: U203.B12 (PT71A)
- new net SDRAM.A5: U203.A12 (PT76A)
- new net SDRAM.A6: U203.B13 (PT78A)
- new net SDRAM.A7: U203.A13 (PT76B)
- new net SDRAM.A8: U203.A14 (PT83A)
- new net SDRAM.A9: U203.A18 (PT119A)
- new net SDRAM.BA0: U203.B15 (PT105A)
- new net SDRAM.BA1: U203.A15 (PT103A)
- new net SDRAM.CKE: U203.B19 (PT119B)
- new net SDRAM.CLK: U203.B20 (PT121B)
- new net SDRAM.DQ0: U203.F18 (PR14D)
- new net SDRAM.DQ1: U203.E18 (PR14C)
- new net SDRAM.DQ10: U203.G20 (PR38D)
- new net SDRAM.DQ11: U203.G19 (PR41A)
- new net SDRAM.DQ12: U203.H20 (PR41B)
- new net SDRAM.DQ13: U203.J20 (PR44C)
- new net SDRAM.DQ14: U203.K19 (PR44B)
- new net SDRAM.DQ15: U203.K20 (PR44D)
- new net SDRAM.DQ2: U203.D18 (PR14A)
- new net SDRAM.DQ3: U203.E19 (PR35D)
- new net SDRAM.DQ4: U203.E20 (PR38A)
- new net SDRAM.DQ5: U203.D19 (PR35B)
- new net SDRAM.DQ6: U203.D20 (PR35C)
- new net SDRAM.DQ7: U203.E17 (PR14B)
- new net SDRAM.DQ8: U203.F20 (PR38C)
- new net SDRAM.DQ9: U203.F19 (PR38B)
- new net SDRAM.DQMH: U203.C20 (PR35A)
- new net SDRAM.DQML: U203.E16 (PR11C)
- new net SDRAM.~{CAS}: U203.A17 (PT116A)
- new net SDRAM.~{CS}: U203.A16 (PT110A)
- new net SDRAM.~{RAS}: U203.B16 (PT110B)
- new net SDRAM.~{WE}: U203.B17 (PT114A)
- new net UART1.RX: U203.T16 (PR77A)
- new net UART1.TX: U203.U16 (PR92C)
- new net UART2.RX: U203.R16 (PR56C)
- new net UART2.TX: U203.N16 (PR53A)
- new net UC_GPIO0: U203.L5 (PL56D)
- new net UC_GPIO1: U203.N2 (PL89A)
- new net ULPI.CLKOUT: U203.L20 (PR47A)
- new net ULPI.D0: U203.U19 (PR89C)
- new net ULPI.D1: U203.U20 (PR86D)
- new net ULPI.D2: U203.T19 (PR89A)
- new net ULPI.D3: U203.T20 (PR86C)
- new net ULPI.D4: U203.R20 (PR86B)
- new net ULPI.D5: U203.P19 (PR83C)
- new net ULPI.D6: U203.P20 (PR86A)
- new net ULPI.D7: U203.N19 (PR83A)
- new net ULPI.DIR: U203.M19 (PR47D)
- new net ULPI.NXT: U203.M20 (PR47B)
- new net ULPI.RESET: U203.L19 (PR47C)
- new net ULPI.STP: U203.N20 (PR83B)
- new net _HDMI_CK+: C208.2, J201.10 (CK+)
- new net _HDMI_CK-: C207.2, J201.12 (CK-)
- new net _HDMI_D0+: C206.2, J201.7 (D0+)
- new net _HDMI_D0-: C205.2, J201.9 (D0-)
- new net _HDMI_D1+: C204.2, J201.4 (D1+)
- new net _HDMI_D1-: C203.2, J201.6 (D1-)
- new net _HDMI_D2+: C201.2, J201.1 (D2+)
- new net _HDMI_D2-: C202.2, J201.3 (D2-)
- new net ~{INIT}: R204.2, U203.V3 (~{INIT})
- new net ~{PROGRAM}: R205.2, U203.W3 (~{PROGRAM})
Other:
- note added: "CLK"
- note added: "FPGA Config"
- note added: "IO Header"
- note added: "LEDs"
- note added: "PCLKT3_1"
- note added: "Power"
- note added: "SD Card"
- moved on the sheet: C1, C301, C302, C303, C304, C305, C306, C307, C308, C309, C310, C311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
